File: board/HispalisFPGA.kicad_pcb (KiCad board)
At the start: 6 copper layers, 17.8 x 61 mm, 95 parts, among them J1 Conn_02x03_Odd_Even, J2 Micro_SD_Card_Det_Hirose_DM3AT, J3 USBC, J4 Conn_01x24, J5 Conn_01x24, J6 Conn_02x09_Odd_Even, SW1 SW_Push, U1 LFE5UM-285, U10 PUSB3FR4Z, U11 PUSB3FR4Z, U2 S27KS0641DPBHI020, U3 DSC6001CI2A-016.0000T, U4 FAN53555, U5 MIC5504-2.5YMT-TR, U6 Conn_02x03_Counter_Clockwise, U7 FAN53600, U8 S25FL064L, U9 MIC5504-1.2YMT-TR

Commit message: Regenerate PCB layout file
Parts:
- removed C44, C45, C46, C47: 100nF, Footprints:C_0201_NoSilk
- removed D1, D2: LED, LEDs:LED_0603
- removed J1: Conn_02x03_Odd_Even, Pin_Headers:Pin_Header_Straight_2x03_Pitch1.00mm_SMD
- removed J2: Micro_SD_Card_Det_Hirose_DM3AT, Footprints:DM3D-SF
- removed J3: USBC, tinyfpga_boards:USBC_DX07S024JJ2R1300
- removed J4, J5: Conn_01x24, Pin_Headers:Pin_Header_Straight_1x24_Pitch2.54mm
- removed J6: Conn_02x09_Odd_Even, Pin_Headers:Pin_Header_Straight_2x11_Pitch2.54mm_SMD
- removed REF** (x4): , Footprints:R_0603_HandSoldering
- removed REF** (x3): Fiducial, Footprints:Fiducial
- removed REF***: OSHW-Logo_5.7x6mm_SilkScreen, Symbols:OSHW-Logo_5.7x6mm_SilkScreen
- removed TP11, TP12 (x9), TP13: TEST, Footprints:small-testpoint
- removed U1: LFE5UM-285, Footprints:csfBGA 285
- removed U10, U11: PUSB3FR4Z, Footprints:PUSB3FR4Z
- removed U2: S27KS0641DPBHI020, Footprints:FBGA-24
- removed U3: DSC6001CI2A-016.0000T, Footprints:DSC6001HI2A
- removed U4: FAN53555, Footprints:WLCSP-20
- removed U5: MIC5504-2.5YMT-TR, Footprints:Thin-DFN4
- removed U6: Conn_02x03_Counter_Clockwise, Footprints:ASG2-D-X-B
- removed U7: FAN53600, Footprints:WLCSP-6
- removed U8: S25FL064L, Housings_SOIC:SOIJ-8_5.3x5.3mm_Pitch1.27mm
- removed U9: MIC5504-1.2YMT-TR, Footprints:Thin-DFN4
- added 1V1_SW_REG1: TPS565208, Package_TO_SOT_SMD:SOT-23-6, F.Cu at (172.3, 94.8)
- added 2V5_LDO_REG1: TLV73325PDBVR, Package_TO_SOT_SMD:SOT-23-5, F.Cu at (172.3, 99.4)
- added 3V3_SW_REG1: TPS63001DRCR, Package_SON:Texas_DRC0010J_ThermalVias, F.Cu at (155.2, 134.2)
- added 5V_LINE1: Conn_01x02_Socket, Connector_PinSocket_2.54mm:PinSocket_1x02_P2.54mm_Vertical, F.Cu at (172.1, 103.9)
- added BLED1: LED, LED_SMD:LED_0603_1608Metric, F.Cu at (156.7, 104.6)
- added BLED2: LED, LED_SMD:LED_0603_1608Metric, F.Cu at (156.7, 107.2)
- added BTN1: SW_Push, Button_Switch_THT:SW_PUSH_6mm, F.Cu at (135.7, 87.6)
- added BTN2: SW_Push, Button_Switch_THT:SW_PUSH_6mm, F.Cu at (135.7, 96.2)
- added BTN3: SW_Push, Button_Switch_THT:SW_PUSH_6mm, F.Cu at (135.7, 104.7)
- added BTN4: SW_Push, Button_Switch_THT:SW_PUSH_6mm, F.Cu at (135.7, 113.3)
- added BTN5: SW_Push, Button_Switch_THT:SW_PUSH_6mm, F.Cu at (135.7, 121.8)
- added BTN6: SW_Push, Button_Switch_THT:SW_PUSH_6mm, F.Cu at (135.7, 130.4)
- added C21: 100nF, Capacitor_SMD:C_0402_1005Metric, F.Cu at (159.0, 98.4)
- added C25: 1uF, Capacitor_SMD:C_0402_1005Metric, F.Cu at (161.9, 86.6)
- added C27: 100nF, Capacitor_SMD:C_0402_1005Metric, F.Cu at (161.9, 88.5)
- added C32: 100nF, Capacitor_SMD:C_0402_1005Metric, F.Cu at (161.9, 98.4)
- added CLK1: ASEDV-16.000MHZ-LR-T, Oscillator:Oscillator_SMD_Abracon_ASE-4Pin_3.2x2.5mm, F.Cu at (160.2, 133.9)
- added CLK2: SWPM201DCAIAB-200.000000, Oscillator:Oscillator_SMD_SiTime_PQFD-6L_3.2x2.5mm, F.Cu at (160.9, 105.8)
- added DISPLAY1: MHDC3641SRBW, Display_7Segment:CA56-12SRWA, F.Cu at (115.8, 105.2)
- added ESD1: ESD9B5.0ST5G, Diode_SMD:D_SOD-923, F.Cu at (164.4, 104.3)
- added ESD2: TPD6S300A, Package_DFN_QFN:WQFN-20-1EP_3x3mm_P0.4mm_EP1.7x1.7mm_ThermalVias, F.Cu at (167.0, 133.5)
- added ESD3: DT1240A-08LP3810, Package_DFN_QFN:UDFN-9_1.0x3.8mm_P0.5mm, F.Cu at (150.5, 134.7)
- added FB1: 100MHz, Inductor_SMD:L_0603_1608Metric, F.Cu at (150.7, 128.1)
- added FB2: 100MHz, Inductor_SMD:L_0603_1608Metric, F.Cu at (150.7, 130.6)
- added FLASH1: W25Q128JVS, Package_SO:SOIC-8_5.23x5.23mm_P1.27mm, F.Cu at (171.3, 89.0)
- added FPGA1: LFE5UM-285, Footprints:csfBGA 285, F.Cu at (169.9, 114.8)
- added JTAG1: Conn_02x03_Odd_Even, Connector_PinSocket_2.54mm:PinSocket_2x03_P2.54mm_Vertical_SMD, F.Cu at (169.4, 126.0)
- added LD1: LED, LED_SMD:LED_0805_2012Metric, F.Cu at (146.5, 110.8)
- added LD2: LED, LED_SMD:LED_0805_2012Metric, F.Cu at (146.5, 113.8)
- added LD3: LED, LED_SMD:LED_0805_2012Metric, F.Cu at (146.5, 116.8)
- added LD4: LED, LED_SMD:LED_0805_2012Metric, F.Cu at (146.5, 119.9)
- added LD5: LED, LED_SMD:LED_0805_2012Metric, F.Cu at (146.5, 122.9)
- added LD6: LED, LED_SMD:LED_0805_2012Metric, F.Cu at (146.5, 126.0)
- added LD7: LED, LED_SMD:LED_0805_2012Metric, F.Cu at (146.5, 129.0)
- added LD8: LED, LED_SMD:LED_0805_2012Metric, F.Cu at (146.5, 132.0)
- added PMOD1: Conn_02x06_Top_Bottom, Connector_PinSocket_2.54mm:PinSocket_2x06_P2.54mm_Horizontal, F.Cu at (126.4, 70.6)
- added PMOD2: Conn_02x06_Top_Bottom, Connector_PinSocket_2.54mm:PinSocket_2x06_P2.54mm_Horizontal, F.Cu at (142.3, 70.6)
- added PMOD3: Conn_02x06_Top_Bottom, Connector_PinSocket_2.54mm:PinSocket_2x06_P2.54mm_Horizontal, F.Cu at (158.2, 70.6)
- added PMOD4: Conn_02x06_Top_Bottom, Connector_PinSocket_2.54mm:PinSocket_2x06_P2.54mm_Horizontal, F.Cu at (174.1, 70.6)
- added Q1: DMG1012T, Package_TO_SOT_SMD:SOT-523, F.Cu at (168.1, 93.9)
- added Q2: DMG1012T, Package_TO_SOT_SMD:SOT-523, F.Cu at (168.1, 97.1)
- added Q3: DMG1012T, Package_TO_SOT_SMD:SOT-523, F.Cu at (168.1, 100.2)
- added Q4: DMG1012T, Package_TO_SOT_SMD:SOT-523, F.Cu at (168.1, 103.4)
- added R1: 100R, Resistor_SMD:R_0402_1005Metric, F.Cu at (154.2, 110.2)
- added R14: 4.7K, Resistor_SMD:R_0402_1005Metric, F.Cu at (160.0, 112.2)
- added R15: 4.7K, Resistor_SMD:R_0402_1005Metric, F.Cu at (160.0, 114.2)
- added R16: 4.7K, Resistor_SMD:R_0402_1005Metric, F.Cu at (160.0, 116.2)
- added R17: 10K, Resistor_SMD:R_0402_1005Metric, F.Cu at (160.0, 118.2)
- added R18: 10K, Resistor_SMD:R_0402_1005Metric, F.Cu at (160.0, 120.2)
- added R19: 10K, Resistor_SMD:R_0402_1005Metric, F.Cu at (162.9, 110.2)
- added R2: 10K, Resistor_SMD:R_0402_1005Metric, F.Cu at (154.2, 112.2)
- added R20: 10K, Resistor_SMD:R_0402_1005Metric, F.Cu at (162.9, 112.2)
- added R21: 10K, Resistor_SMD:R_0402_1005Metric, F.Cu at (162.9, 114.2)
- added R22: 4.7K, Resistor_SMD:R_0402_1005Metric, F.Cu at (162.9, 116.2)
- added R23: 1.5K, Resistor_SMD:R_0402_1005Metric, F.Cu at (162.9, 118.2)
- added R9: 10K, Resistor_SMD:R_0402_1005Metric, F.Cu at (157.1, 114.2)
- added TP2: TEST, TestPoint:TestPoint_Pad_D1.0mm, F.Cu at (176.0, 125.8)
- added TP3: TEST, TestPoint:TestPoint_Pad_D1.0mm, F.Cu at (176.0, 128.8)
- added USB_C1: MOLEX-105450-0101, Connector_USB:USB_C_Receptacle_Molex_105450-0101, F.Cu at (158.5, 126.2)
- C1: value 1uF -> 100nF; footprint Footprints:C_0402_NoSilk -> Capacitor_SMD:C_0402_1005Metric; moved to F.Cu
- C10, C15, C30, C34, C6: footprint Footprints:C_0201_NoSilk -> Capacitor_SMD:C_0402_1005Metric; moved to F.Cu
- C11, C12, C31, C35: value 10nf -> 100nF; footprint Footprints:C_0201_NoSilk -> Capacitor_SMD:C_0402_1005Metric; moved to F.Cu
- C13, C28, C3, C39, C41, C9: value 100nF -> 10nF; footprint Footprints:C_0201_NoSilk -> Capacitor_SMD:C_0402_1005Metric; moved to F.Cu
- C14, C16: value 10nf -> 10nF; footprint Footprints:C_0201_NoSilk -> Capacitor_SMD:C_0402_1005Metric; moved to F.Cu
- C17, C42, C43: value 1uF -> 100nF; footprint Footprints:C_0402_NoSilk -> Capacitor_SMD:C_0402_1005Metric
- C18: value 100nF -> 10uF; footprint Footprints:C_0201_NoSilk -> Capacitor_SMD:C_0603_1608Metric; moved to F.Cu
- C19: value 2.2uF -> 10nF; footprint Footprints:C_0402_NoSilk -> Capacitor_SMD:C_0402_1005Metric
- C2: footprint Footprints:C_0402_NoSilk -> Capacitor_SMD:C_0402_1005Metric; moved to F.Cu
- C20: value 1uF -> 10uF; footprint Footprints:C_0402_NoSilk -> Capacitor_SMD:C_0603_1608Metric
- C22: value 22uF -> 100nF; footprint Capacitors_SMD:C_0603 -> Capacitor_SMD:C_0402_1005Metric
- C23: value 10uF -> 22uF; footprint Capacitors_SMD:C_0603 -> Capacitor_SMD:C_0603_1608Metric
- C24: value 100nF -> 10nF; footprint Footprints:C_0201_NoSilk -> Capacitor_SMD:C_0402_1005Metric
- C26: value 100nF -> 22uF; footprint Footprints:C_0201_NoSilk -> Capacitor_SMD:C_0603_1608Metric
- C29: value 100nF -> 1uF; footprint Footprints:C_0201_NoSilk -> Capacitor_SMD:C_0402_1005Metric; moved to F.Cu
- C33: value 10uF -> 100nF; footprint Capacitors_SMD:C_0603 -> Capacitor_SMD:C_0402_1005Metric; moved to F.Cu
- C36: value 1nF -> 100nF; footprint Footprints:C_0201_NoSilk -> Capacitor_SMD:C_0402_1005Metric; moved to F.Cu
- C37: footprint Capacitors_SMD:C_0201_NoSilk -> Capacitor_SMD:C_0402_1005Metric; moved to F.Cu
- C38: value 10nF -> 1nF; footprint Footprints:C_0201_NoSilk -> Capacitor_SMD:C_0402_1005Metric; moved to F.Cu
- C4, C7: value 10nf -> 10uF; footprint Footprints:C_0201_NoSilk -> Capacitor_SMD:C_0603_1608Metric; moved to F.Cu
- C40: value 10nF -> 100nF; footprint Footprints:C_0201_NoSilk -> Capacitor_SMD:C_0402_1005Metric; moved to F.Cu
- C5: footprint Capacitors_SMD:C_0603 -> Capacitor_SMD:C_0603_1608Metric
- C8: value 10nF -> 100nF; footprint Footprints:C_0201_NoSilk -> Capacitor_SMD:C_0402_1005Metric
- L1: value 330nH -> 2.2uH; footprint Inductors_SMD:L_0805 -> Inductor_SMD:L_0805_2012Metric
- L2: value 1uH -> 2.2uH; footprint Inductors_SMD:L_0805 -> Inductor_SMD:L_0805_2012Metric
- R10, R4: value 4.7k -> 10K; footprint Footprints:R_0402_NoSilk -> Resistor_SMD:R_0402_1005Metric
- R11: value 1.5k -> 10K; footprint Footprints:R_0402_NoSilk -> Resistor_SMD:R_0402_1005Metric; moved to F.Cu
- R12: value 4.7K -> 10K; footprint Footprints:R_0402_NoSilk -> Resistor_SMD:R_0402_1005Metric
- R13: footprint Footprints:R_0402_NoSilk -> Resistor_SMD:R_0402_1005Metric
- R3: value 0 -> 12K; footprint Footprints:R_0201_NoSilk -> Resistor_SMD:R_0402_1005Metric
- R5, R7: value 4.7k -> 10K; footprint Footprints:R_0201_NoSilk -> Resistor_SMD:R_0402_1005Metric; moved to F.Cu
- R6: value 100K -> 10K; footprint Footprints:R_0402_NoSilk -> Resistor_SMD:R_0402_1005Metric; moved to F.Cu
- R8: value 0 -> 10K; footprint Footprints:R_0201_NoSilk -> Resistor_SMD:R_0402_1005Metric
- SW1: value SW_Push -> SW_DIP_x08; footprint Footprints:PTS_810_SMT_Switch -> Button_Switch_SMD:SW_DIP_SPSTx08_Slide_6.7x21.88mm_W6.73mm_P2.54mm_LowProfile_JPin
- TP1: footprint Footprints:small-testpoint -> TestPoint:TestPoint_Pad_D1.0mm; moved to F.Cu
- moved L1 79.7 mm to (171.9, 132.2), turned to 0 degrees
- moved L2 78.4 mm to (171.9, 135.0)
- moved C23 62.9 mm to (150.7, 123.0), turned to 0 degrees
- moved TP1 62.3 mm to (176.0, 122.7)
- moved C5 55.5 mm to (150.7, 113.0)
- moved R3 55.0 mm to (154.2, 114.2), turned to 0 degrees
- moved R8 54.7 mm to (157.1, 112.2), turned to 0 degrees
- moved C20 54.4 mm to (150.7, 120.5)
- moved R4 54.2 mm to (154.2, 116.2)
- moved R11 50.8 mm to (157.1, 118.2), turned to 0 degrees
- moved R5 47.5 mm to (154.2, 118.2)
- moved C22 44.1 mm to (159.0, 100.4)
- moved R7 42.3 mm to (157.1, 110.2), turned to 0 degrees
- moved C19 41.0 mm to (159.0, 96.4)
- moved C8 40.2 mm to (156.1, 94.5)
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Connections:
- C10 pad 1: +1V1 -> VCCIO0
- C11 pad 1: VCCIO0 -> GND
- C11 pad 2: GND -> Net-(3V3_SW_REG1-EN)
- C12 pad 1: +1V1 -> FPGA_PWR
- C13 pad 1: +1V1 -> VCCIO0
- C14 pad 1: +1V1 -> FPGA_PWR
- C15 pad 1: +1V1 -> FPGA_PWR
- C16 pad 1: +1V1 -> FPGA_PWR
- C19 pad 1: +5V -> VCCIO0
- C2 pad 1: VCCIO0 -> +2V5
- C20 pad 1: +2V5 -> VCCIO0
- C22 pad 1: +1V1 -> VCCIO0
- C23 pad 1: VCCIO0 -> FPGA_PWR
- C26 pad 1: VCCIO0 -> FPGA_PWR
- C29 pad 1: VCCIO0 -> +2V5
- C3 pad 1: VCCIO0 -> +2V5
- C31 pad 1: VCCIO0 -> Net-(USB_C1-SHIELD)
- C33 pad 1: VCCIO0 -> CH0_TX-
- C33 pad 2: GND -> Net-(USB_C1-TX1-)
- C34 pad 1: VCCIO0 -> Net-(USB_C1-TX2+)
- C34 pad 2: GND -> CH1_TX+
- C35 pad 1: VCCIO0 -> CH0_TX+
- C35 pad 2: GND -> Net-(USB_C1-TX1+)
- C36 pad 1: +1V2A -> Net-(USB_C1-TX2-)
- C36 pad 2: GND -> CH1_TX-
- C37 pad 1: +1V2A -> FPGA_PWR
- C38 pad 1: +1V2A -> FPGA_PWR
- C39 pad 1: +1V2A -> FPGA_PWR
- C4 pad 1: VCCIO0 -> +5V
- C40 pad 1: +1V2A -> FPGA_PWR
- C41 pad 1: +1V2A -> FPGA_PWR
- C42 pad 1: VCCIO0 -> FPGA_PWR
- C43 pad 1: +1V2A -> Net-(ESD2-VBIAS)
- C6 pad 1: +2V5 -> FPGA_PWR
- C7 pad 1: +2V5 -> +5V
- C9 pad 1: VCCIO0 -> FPGA_PWR
- L1 pad 2: +1V1 -> Net-(3V3_SW_REG1-L1)
- L2 pad 2: VCCIO0 -> FPGA_PWR
- R10 pad 1: VCCIO0 -> SW7
- R10 pad 2: PROGRAMN -> GND
- R11 pad 1: USB_CONNECT -> SW8
- R11 pad 2: USB_D+ -> GND
- R12 pad 1: Net-(D1-Pad1) -> VCCIO0
- R12 pad 2: GND -> PROGRAMN
- R13 pad 1: Net-(D2-Pad1) -> CFG_MODE_SEL_0
- R3 pad 1: +5V -> Net-(1V1_SW_REG1-VFB)
- R3 pad 2: Net-(R3-Pad2) -> GND
- R4 pad 1: TCK -> SW1
- R5 pad 1: VCCIO0 -> SW2
- R5 pad 2: CFG_MODE_SEL_1 -> GND
- R6 pad 1: SDCARD_DET -> SW3
- R7 pad 1: CFG_MODE_SEL_0 -> SW4
- R8 pad 1: Net-(R3-Pad2) -> SW5
- SW1 pad 1: GND -> SW1
- SW1 pad 2: PROGRAMN -> SW2
- TP1 pad 1: +1V2A -> FPGA_PWR
Routing:
- net GND: track 163.3 -> 0.00 mm, vias 65 -> 0
- net VCCIO0: track 68.0 -> 0.00 mm, vias 23 -> 0
- net PROGRAMN: track 47.5 -> 0.00 mm, vias 4 -> 0
- net SDCARD_DAT3_CD: track 35.7 -> 0.00 mm, vias 3 -> 0
- net SDCARD_DAT0: track 34.9 -> 0.00 mm, vias 2 -> 0
- net SDCARD_DAT1: track 33.8 -> 0.00 mm, vias 2 -> 0
- net PIN23: track 33.8 -> 0.00 mm
- net SDCARD_CMD: track 33.7 -> 0.00 mm, vias 2 -> 0
- net PIN22: track 33.5 -> 0.00 mm
- net SDCARD_DAT2: track 33.1 -> 0.00 mm, vias 3 -> 0
- net SDCARD_CLK: track 32.4 -> 0.00 mm, vias 3 -> 0
- net USB_D+: track 32.1 -> 0.00 mm, vias 2 -> 0
- net PIN24: track 31.7 -> 0.00 mm
- net USB_D-: track 31.5 -> 0.00 mm, vias 3 -> 0
- net PIN42: track 31.0 -> 0.00 mm, vias 1 -> 0
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- removed copper zone on F.Cu, net +1V1
- removed copper zone on PWR.Cu, net +1V1
- removed copper zone on B.Cu, net +1V2A
- removed copper zone on F.Cu, net +1V2A
- removed copper zone on PWR.Cu, net +1V2A
- removed copper zone on F.Cu, net +2V5
- removed copper zone on F.Cu, net +5V
- removed copper zone on PWR.Cu, net +5V
- removed copper zone on B.Cu, net GND
- removed copper zone on B_GND.Cu, net GND
- removed copper zone on F.Cu, net GND
- removed copper zone on F_GND.Cu, net GND
- removed copper zone on F.Cu, net Net-(1V1_SW_REG1-SW)
- removed copper zone on F.Cu, net Net-(3V3_SW_REG1-L2)
- removed copper zone on F.Cu, net VCCIO0
- removed copper zone on PWR.Cu, net VCCIO0
Other:
- board outline removed
- copper layers 6 -> 2
- net class BGA-Power removed
- net class BGA-Signal removed
- net class Default removed
- net class Power removed
- net class USB3 removed
- rule pad_to_mask_clearance: 0.05 -> 0
- board text removed: "1"
- board text removed: "10"
- board text removed: "11"
- board text removed: "12"
- board text removed: "13"
- board text removed: "14"
- board text removed: "15"
- board text removed: "16"
- board text removed: "17"
- board text removed: "18"
- board text removed: "19"
- board text removed: "2"
- board text removed: "20"
- board text removed: "21"
- board text removed: "22"
- board text removed: "23"
- board text removed: "24"
- board text removed: "25"
- board text removed: "26"
- board text removed: "27"
- board text removed: "28"
- board text removed: "29"
- board text removed: "3"
- board text removed: "30"
- board text removed: "31"
- board text removed: "32"
- board text removed: "33"
- board text removed: "34"
- board text removed: "36"
- board text removed: "37"
- board text removed: "38"
- board text removed: "39"
- board text removed: "3v"
- board text removed: "3v3"
- board text removed: "4"
- board text removed: "40"
- board text removed: "41"
- board text removed: "42"
- board text removed: "43"
- board text removed: "44"
- board text removed: "45"
- board text removed: "46"
- board text removed: "47"
- board text removed: "48"
- board text removed: "49"
- board text removed: "50"
- board text removed: "51"
- board text removed: "52"
- board text removed: "53"
- board text removed: "54"
- board text removed: "55"
- board text removed: "6"
- board text removed: "7"
- board text removed: "8"
- board text removed: "9"
- board text removed: "BANK0"
- board text removed: "BANK1"
- board text removed: "BANK2"
- board text removed: "BANK3"
- board text removed: "BANK6"
- board text removed: "BANK7"
- board text removed: "BANK8"
- board text removed: "CLK"
- board text removed: "CMD"
- board text removed: "D0"
- board text removed: "D1"
- board text removed: "D2"
- board text removed: "D3"
- board text removed: "DET"
- board text removed: "EX"
- board text removed: "G"
- board text removed: "GND"
- board text removed: "TinyFPGA"
- board text removed: "Vin"
