File: board/ecp5-aux-connections.kicad_sch (KiCad schematic)
At the start: 15 parts

Commit message: Complete schematic
Parts:
- removed unit 11 of FPGA1
- removed unit 10 of FPGA1
- FPGA1: value LFE5UM-381 -> LFE5U-25F; symbol FPGA_Lattice:LFE5UM-85F-6BG381x -> FPGA_Lattice:LFE5U-85F-8BG381x; JLC (none) -> CABGA-381; LCSC (none) -> C1550939
- renumbered C51 to C45, C52 to C46
Connections:
- no-connect marks 21 -> 1
Other:
- note removed: "FPGA Bitstream Configuration"
- note removed: "SERDES"
- moved on the sheet: BLED1, BLED2, BOOT_BTN1, C45, C46, CLK1, FLASH1, FPGA1I, R29, R30, R31, R32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
