File: board/connectors.kicad_sch (KiCad schematic)
At the start: 18 parts, among them J1 HC-TYPE-C-16P-01A

Commit message: Complete schematic
Parts:
- renumbered C27 to C21, C28 to C22
Connections:
- no-connect marks 7 -> 9
Changed lines of the file:
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@@
 	)
 	(no_connect
+		(at 119.38 146.05)
+	)
+	(no_connect
 		(at 147.32 66.04)
 	)
@@
 	)
 	(no_connect
+		(at 119.38 143.51)
+	)
+	(no_connect
 		(at 100.33 78.74)
 	)
@@
 		(on_board yes)
 		(dnp no)
-		(property "Reference" "C27"
+		(property "Reference" "C21"
 			(at 77.978 88.138 0)
 			(effects
@@
 			(project "HispalisFPGA"
 				(path "/864346d0-d3ef-428e-a44f-9476f195db98/b6a4d967-b3aa-4b5c-a3fd-3675ad6e05ec"
-					(reference "C27")
+					(reference "C21")
 					(unit 1)
 				)
@@
 		(on_board yes)
 		(dnp no)
-		(property "Reference" "C28"
+		(property "Reference" "C22"
 			(at 150.368 75.692 0)
 			(effects
@@
 			(project "HispalisFPGA"
 				(path "/864346d0-d3ef-428e-a44f-9476f195db98/b6a4d967-b3aa-4b5c-a3fd-3675ad6e05ec"
-					(reference "C28")
+					(reference "C22")
 					(unit 1)
 				)
