File: board/ecp5-io-connections.kicad_sch (KiCad schematic)
At the start: 9 parts

Commit message: Add metadata
Other:
- title: HispalisFPGA FPGA I/O Connections -> HispalisFPGA ECP5 I/O Connections
Changed lines of the file:
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@@
 	(paper "A4" portrait)
 	(title_block
-		(title "HispalisFPGA FPGA I/O Connections")
+		(title "HispalisFPGA ECP5 I/O Connections")
 		(date "2024-10-21")
 		(rev "A")
