File: board/ports.kicad_sch (KiCad schematic)
At the start: 18 parts, among them J1 HC-TYPE-C-16P-01A

Commit message: Add metadata
Other:
- title: HispalisFPGA - Ports -> HispalisFPGA Ports
Changed lines of the file:
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@@
 	(paper "A4" portrait)
 	(title_block
-		(title "HispalisFPGA - Ports")
+		(title "HispalisFPGA Ports")
 		(date "2024-10-21")
 		(rev "A")
