File: board/ports.kicad_sch (KiCad schematic)
At the start: 18 parts, among them J1 HC-TYPE-C-16P-01A

Commit message: Change JTAG pin header parts reference
Parts:
- JTAG1: LCSC C6332201 -> C5156616
Changed lines of the file:
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@@
 			)
 		)
-		(property "LCSC" "C6332201"
+		(property "LCSC" "C5156616"
 			(at 124.46 143.51 0)
 			(effects
