File: board/ecp5-io-pins-2.kicad_sch (KiCad schematic)
At the start: 9 parts

Commit message: Change LFE5U chip from BGA381 to BGA256 package
Parts:
- removed U3: ~, HispalisFPGA:CABGA-256_L14.0-W14.0-R16-C16-P0.80-TL, symbol LFE5U-45F-7BG256I:LFE5U-45F-7BG256I
- added FPGA1: LFE5U-45F-7BG256I, HispalisFPGA:CABGA-256_L14.0-W14.0-R16-C16-P0.80-TL, symbol LFE5U-45F-7BG256I:LFE5U-45F-7BG256I
- C37, C43: value 100nF -> 10nF; LCSC C1525 -> C15195
- C38, C40: value 10nF -> 100nF; LCSC C15195 -> C1525
Connections:
- net +3V3: now also FPGA1.H6 (VCCIO7), FPGA1.H7 (VCCIO7), FPGA1.J6 (VCCIO6), FPGA1.J7 (VCCIO6), FPGA1.K11 (VCCIO3), FPGA1.L11 (VCCIO3), FPGA1.L6 (VCCIO8)
- net BTN1: now also FPGA1.J4 (PL26C)
- net BTN2: now also FPGA1.K4 (PL38A/GR_PCLK6_0)
- net BTN3: now also FPGA1.T15 (PR59D)
- net BTN4: now also FPGA1.L3 (PL41C)
- net BTN5: now also FPGA1.K3 (PL29D)
- net CFG_0: now also FPGA1.N10 (CFG_0)
- net CFG_1: now also FPGA1.P10 (CFG_1)
- net CFG_2: now also FPGA1.R10 (CFG_2)
- net CSSPIN: now also FPGA1.N8 (PB15A/HOLDN/DI/BUSY/CSSPIN/CEN)
- net DISPLAY_D2: now also FPGA1.C3 (PL11C)
- net DISPLAY_D3: now also FPGA1.D3 (PL11D)
- net DISPLAY_SB: now also FPGA1.C2 (PL14B)
- net DISPLAY_SC: now also FPGA1.B2 (PL11B/ULC_GPLL0C_IN)
- net DISPLAY_SF: now also FPGA1.B1 (PL11A/ULC_GPLL0T_IN)
- net DISPLAY_SG: now also FPGA1.C1 (PL14A)
- net DONE: now also FPGA1.P9 (DONE)
- net IO2: now also FPGA1.M7 (PB9B/D2/IO2)
- net IO3: now also FPGA1.N7 (PB9A/D3/IO3)
- net LED1: now also FPGA1.J2 (PL32B/PCLKC7_1)
- net LED2: now also FPGA1.K1 (PL32C/PCLKT7_0)
- net LED3: now also FPGA1.K2 (PL32D/PCLKC7_0)
- net LED4: now also FPGA1.L1 (PL35A/PCLKT6_1)
- net LED5: now also FPGA1.L2 (PL35B/PCLKC6_1)
- net LED6: now also FPGA1.M1 (PL35C/PCLKT6_0)
- net LED7: now also FPGA1.M2 (PL35D/PCLKC6_0)
- net LED8: now also FPGA1.N1 (PL41A)
- net MISO: now also FPGA1.T7 (PB11A/D1/MISO/IO1)
- net MOSI: now also FPGA1.T8 (PB11B/D0/MOSI/IO0)
- net PMOD3_1: now also FPGA1.M6 (PL68A)
- net PMOD3_10: now also FPGA1.N3 (PL44D)
- net PMOD3_2: now also FPGA1.M5 (PL65C)
- net PMOD3_3: now also FPGA1.M4 (PL44C)
- net PMOD3_4: now also FPGA1.P3 (PL59B)
- net PMOD3_7: now also FPGA1.N6 (PL68B)
- net PMOD3_8: now also FPGA1.N5 (PL65D)
- net PMOD3_9: now also FPGA1.N4 (PL59A)
- net PMOD4_1: now also FPGA1.R4 (PL62C)
- net PMOD4_10: now also FPGA1.P1 (PL44A)
- net PMOD4_2: now also FPGA1.R3 (PL62B)
- net PMOD4_3: now also FPGA1.R2 (PL59C)
- net PMOD4_4: now also FPGA1.P2 (PL41B)
- net PMOD4_7: now also FPGA1.T4 (PL65B)
- net PMOD4_8: now also FPGA1.T3 (PL62D)
- net PMOD4_9: now also FPGA1.R1 (PL44B/VREF1_6)
- net PROGRAMN: now also FPGA1.R9 (PROGRAMN)
- net SCK: now also FPGA1.N9 (CCLK/MCLK/SCK)
- net SW1: now also FPGA1.D1 (PL17A)
- net SW2: now also FPGA1.E2 (PL17B)
- net SW3: now also FPGA1.E1 (PL20D)
- net SW4: now also FPGA1.F2 (PL20C)
- net SW5: now also FPGA1.F1 (PL23A)
- net SW6: now also FPGA1.G2 (PL23B)
- net SW7: now also FPGA1.G1 (PL29A/GR_PCLK7_1)
- net SW8: now also FPGA1.J1 (PL32A/PCLKT7_1)
- net TCK: now also FPGA1.T10 (TCK)
- net TDI: now also FPGA1.R11 (TDI)
- net TDO: now also FPGA1.M10 (TDO)
- net TMS: now also FPGA1.T11 (TMS)
- no-connect marks 1 -> 62
Other:
- title: HispalisFPGA ECP5 I/O Pins -> (none)
